Commit message: Updated xacro

File: Planning/Workspaces/bumperbot_ws/src/bumperbot_description/urdf/bumperbot.urdf.xacro (robot description, xacro)
@@ -69,3 +69,16 @@
         <origin rpy = "0 0 0" xyz ="0.04755 0 -0.0275"/>
     </joint>
+    <link name = "can_link">
+        <visual>
+            <origin xyz="-0.033 0.03 0.0" rpy="1.57 0.0 0.0"/>
+            <geometry>
+                <mesh filename = "package://bumperbot_description/meshes/can.STL"/>
+            </geometry>
+        </visual>
+    </link>
+    <joint name = "can_joint" type = "fixed">
+        <parent link = "base_link"/>
+        <child link = "can_link"/>
+        <origin rpy = "0 0 0" xyz ="0 0 0.078"/>
+    </joint>
 </robot>

Commit message: Updated xacro

File: Planning/Workspaces/bumperbot_ws/src/bumperbot_description/urdf/bumperbot.urdf.xacro (robot description, xacro)
@@ -71,5 +71,5 @@
     <link name = "can_link">
         <visual>
-            <origin xyz="-0.033 0.03 0.0" rpy="1.57 0.0 0.0"/>
+            <origin xyz="-0.03 0.03 0.0" rpy="1.57 0.0 0.0"/>
             <geometry>
                 <mesh filename = "package://bumperbot_description/meshes/can.STL"/>

Commit message: Updated URDF

File: Planning/Workspaces/bumperbot_ws/src/bumperbot_description/urdf/bumperbot.urdf.xacro (robot description, xacro)
@@ -3,4 +3,11 @@
     <link name = "base_footprint"></link>
     <link name = "base_link">
+        <inertial>
+            <origin xyz="0 0 0.04" rpy="0.0 0.25 0.3" />
+            <mass value="8.2573504e-01"/>
+            <inertia ixx="2.2124416e-02" ixy="-1.2294101e-04" ixz="3.4938785e-04"
+                    iyy="2.1193702e-02" iyz="-5.0120904e-05"
+                    izz="2.0064271e-02" />
+        </inertial>
         <visual>
             <origin rpy = "0 0 0" xyz = "0 0 0"/>
@@ -9,4 +16,10 @@
             </geometry>
         </visual>
+        <collision>
+                <origin rpy = "0 0 0" xyz = "0 0 0"/>
+                <geometry>
+                    <mesh filename = "package://bumperbot_description/meshes/base_link.STL"/>
+                </geometry>
+        </collision>
     </link>
     <joint name = "base_joint" type = "fixed">
@@ -16,4 +29,11 @@
     </joint>
     <link name = "wheel_right_link">
+        <inertial>
+            <origin xyz="0 -0.014 0" rpy="0 0 0" />
+            <mass value="0.0530086090966721" />
+            <inertia ixx="1.88176298336665E-05" ixy="-4.8444933029987E-10" ixz="1.88163708851143E-08"
+                    iyy="3.11510738647764E-05" iyz="-6.93560663069607E-11"
+                    izz="1.8801969558182E-05" />
+        </inertial>
         <visual>
             <origin rpy = "1.57 0 0" xyz = "0 0 0"/>
@@ -22,4 +42,10 @@
             </geometry>
         </visual>
+        <collision>
+            <origin xyz = "0 -0.015 0" rpy = "1.57 0 0"/>
+            <geometry>
+                <sphere radius = "0.033"/>
+            </geometry>
+        </collision>
     </link>
     <joint name = "wheel_right_joint" type = "continuous">
@@ -30,4 +56,11 @@
     </joint>
         <link name = "wheel_left_link">
+        <inertial>
+            <origin xyz="0 0.014 0" rpy="0 0 0" />
+            <mass value="0.0530086043217644" />
+            <inertia ixx="1.8792911368909E-05"  ixy="3.31256392204584E-10" ixz="-1.14082001662767E-08"
+                    iyy="3.11510738759073E-05" iyz="-3.60499245082192E-10"
+                    izz="1.88266886146847E-05" />
+        </inertial>
         <visual>
             <origin rpy = "-1.57 0 0" xyz = "0 0 0"/>
@@ -36,4 +69,10 @@
             </geometry>
         </visual>
+        <collision>
+            <origin xyz = "0 0.015 0" rpy = "1.57 0 0"/>
+            <geometry>
+                <sphere radius = "0.033"/>
+            </geometry>
+        </collision>
     </link>
     <joint name = "wheel_left_joint" type = "continuous">
@@ -44,4 +83,11 @@
     </joint>
     <link name = "caster_front_link">
+        <inertial>
+            <origin xyz="3.89968128948481E-07 2.40073004698083E-07 0.00219173397061506" rpy="0 0 0" />
+            <mass value="1.44379265037903E-06" />
+            <inertia ixx="7.23075276010246E-11" ixy="-6.10956883467859E-16" ixz="2.22849693525031E-15"
+                    iyy="3.8713793085917E-11"  iyz="2.93909858781952E-15"
+                    izz="1.00967486676306E-10" />
+        </inertial>
         <visual>
             <origin rpy = "0 0 0" xyz = "0 0 0"/>
@@ -50,4 +96,10 @@
             </geometry>
         </visual>
+        <collision>
+            <origin xyz = "0 0 0" rpy = "0 0 0"/>
+            <geometry>
+                <sphere radius = "0.005"/>
+            </geometry>
+        </collision>
     </link>
     <joint name = "caster_front_joint" type = "fixed">
@@ -57,4 +109,11 @@
     </joint>
     <link name = "caster_rear_link">
+        <inertial>
+            <origin xyz="3.8996812895542E-07 2.40073004698083E-07 0.00219173397061509" rpy="0 0 0" />
+            <mass value="1.44379265037902E-06" />
+            <inertia ixx="7.23075276010246E-11" ixy="-6.10956872363424E-16" ixz="2.22849693527207E-15"
+                    iyy="3.87137930859167E-11" iyz="2.939098587861E-15"
+                    izz="1.00967486676306E-10" />
+        </inertial>
         <visual>
             <origin rpy = "0 0 0" xyz = "0 0 0"/>
@@ -63,4 +122,10 @@
             </geometry>
         </visual>
+        <collision>
+            <origin xyz = "0 0 0" rpy = "0 0 0"/>
+            <geometry>
+                <sphere radius = "0.033"/>
+            </geometry>
+        </collision>
     </link>
     <joint name = "caster_rear_joint" type = "fixed">

Commit message: Updated robot description

File: Planning/Workspaces/bumperbot_ws/src/bumperbot_description/urdf/bumperbot.urdf.xacro (robot description, xacro)
@@ -1,152 +1,159 @@
 <?xml version="1.0" encoding="UTF-8"?>
-<robot xmlns:xacro="http://www.ros.org/wiki/xacro" name = "bumperbot">
-    <xacro:arg name = "is_ignition" default = "true"/>
-    <xacro:include filename = "$(find bumperbot_description)/urdf/bumperbot_gazebo.xacro"/>
-    <xacro:include filename = "$(find bumperbot_description)/urdf/bumperbot_ros2_control.xacro"/>
-    <link name = "base_footprint"></link>
-    <link name = "base_link">
+<robot xmlns:xacro="http://www.ros.org/wiki/xacro" name="bumperbot">
+    <xacro:arg name="is_ignition" default="true"/>
+    <xacro:include filename="$(find bumperbot_description)/urdf/bumperbot_gazebo.xacro"/>
+    <xacro:include filename="$(find bumperbot_description)/urdf/bumperbot_ros2_control.xacro"/>
+    <!-- BASE FOOTPRINT -->
+    <link name="base_footprint"/>
+    <!-- BASE LINK -->
+    <link name="base_link">
         <inertial>
-            <origin xyz="0 0 0.04" rpy="0.0 0.25 0.3" />
+            <origin xyz="0 0 0.04" rpy="0.0 0.25 0.3"/>
             <mass value="8.2573504e-01"/>
             <inertia ixx="2.2124416e-02" ixy="-1.2294101e-04" ixz="3.4938785e-04"
-                    iyy="2.1193702e-02" iyz="-5.0120904e-05"
-                    izz="2.0064271e-02" />
+                     iyy="2.1193702e-02" iyz="-5.0120904e-05"
+                     izz="2.0064271e-02"/>
         </inertial>
         <visual>
-            <origin rpy = "0 0 0" xyz = "0 0 0"/>
+            <origin xyz="0 0 0" rpy="0 0 0"/>
             <geometry>
-                <mesh filename = "package://bumperbot_description/meshes/base_link.STL"/>
+                <mesh filename="package://bumperbot_description/meshes/base_link.STL"/>
             </geometry>
         </visual>
         <collision>
-                <origin rpy = "0 0 0" xyz = "0 0 0"/>
-                <geometry>
-                    <mesh filename = "package://bumperbot_description/meshes/base_link.STL"/>
-                </geometry>
+            <origin xyz="0 0 0" rpy="0 0 0"/>
+            <geometry>
+                <mesh filename="package://bumperbot_description/meshes/base_link.STL"/>
+            </geometry>
         </collision>
     </link>
-    <joint name = "base_joint" type = "fixed">
-        <parent link = "base_footprint"/>
-        <child link = "base_link"/>
-        <origin rpy = "0 0 0" xyz = "0 0 0.033"/>
+    <joint name="base_joint" type="fixed">
+        <parent link="base_footprint"/>
+        <child link="base_link"/>
+        <origin xyz="0 0 0.033" rpy="0 0 0"/>
     </joint>
-    <link name = "wheel_right_link">
+    <!-- RIGHT WHEEL -->
+    <link name="wheel_right_link">
         <inertial>
-            <origin xyz="0 -0.014 0" rpy="0 0 0" />
-            <mass value="0.0530086090966721" />
+            <origin xyz="0 -0.014 0" rpy="0 0 0"/>
+            <mass value="0.0530086090966721"/>
             <inertia ixx="1.88176298336665E-05" ixy="-4.8444933029987E-10" ixz="1.88163708851143E-08"
-                    iyy="3.11510738647764E-05" iyz="-6.93560663069607E-11"
-                    izz="1.8801969558182E-05" />
+                     iyy="3.11510738647764E-05" iyz="-6.93560663069607E-11"
+                     izz="1.8801969558182E-05"/>
         </inertial>
         <visual>
-            <origin rpy = "1.57 0 0" xyz = "0 0 0"/>
+            <origin xyz="0 0 0" rpy="1.57 0 0"/>
             <geometry>
-                <mesh filename = "package://bumperbot_description/meshes/wheel_right_link.STL"/>
+                <mesh filename="package://bumperbot_description/meshes/wheel_right_link.STL"/>
             </geometry>
         </visual>
         <collision>
-            <origin xyz = "0 -0.015 0" rpy = "1.57 0 0"/>
+            <origin xyz="0 -0.015 0" rpy="1.57 0 0"/>
             <geometry>
-                <sphere radius = "0.033"/>
+                <sphere radius="0.033"/>
             </geometry>
         </collision>
     </link>
-    <joint name = "wheel_right_joint" type = "continuous">
-        <parent link = "base_link"/>
-        <child link = "wheel_right_link"/>
-        <axis xyz = "0 1 0"/>
-        <origin rpy = "0 0 0" xyz = "0 -0.07 0"/>
+    <joint name="wheel_right_joint" type="continuous">
+        <origin xyz="0 -0.0701101849418637 0" rpy="0 0 0"/>
+        <parent link="base_link"/>
+        <child link="wheel_right_link"/>
+        <axis xyz="0 1 0"/>
     </joint>
-        <link name = "wheel_left_link">
+    <!-- LEFT WHEEL -->
+    <link name="wheel_left_link">
         <inertial>
-            <origin xyz="0 0.014 0" rpy="0 0 0" />
-            <mass value="0.0530086043217644" />
-            <inertia ixx="1.8792911368909E-05"  ixy="3.31256392204584E-10" ixz="-1.14082001662767E-08"
-                    iyy="3.11510738759073E-05" iyz="-3.60499245082192E-10"
-                    izz="1.88266886146847E-05" />
+            <origin xyz="0 0.014 0" rpy="0 0 0"/>
+            <mass value="0.0530086043217644"/>
+            <inertia ixx="1.8792911368909E-05" ixy="3.31256392204584E-10" ixz="-1.14082001662767E-08"
+                     iyy="3.11510738759073E-05" iyz="-3.60499245082192E-10"
+                     izz="1.88266886146847E-05"/>
         </inertial>
         <visual>
-            <origin rpy = "-1.57 0 0" xyz = "0 0 0"/>
+            <origin xyz="0 0 0" rpy="-1.57 0 0"/>
             <geometry>
-                <mesh filename = "package://bumperbot_description/meshes/wheel_left_link.STL"/>
+                <mesh filename="package://bumperbot_description/meshes/wheel_left_link.STL"/>
             </geometry>
         </visual>
         <collision>
-            <origin xyz = "0 0.015 0" rpy = "1.57 0 0"/>
+            <origin xyz="0 0.015 0" rpy="-1.57 0 0"/>
             <geometry>
-                <sphere radius = "0.033"/>
+                <sphere radius="0.033"/>
             </geometry>
         </collision>
     </link>
-    <joint name = "wheel_left_joint" type = "continuous">
-        <parent link = "base_link"/>
-        <child link = "wheel_left_link"/>
-        <axis xyz = "0 1 0"/>
-        <origin rpy = "0 0 0" xyz = "0 0.07 0"/>
+    <joint name="wheel_left_joint" type="continuous">
+        <origin xyz="0 0.0701101849418642 0" rpy="0 0 0"/>
+        <parent link="base_link"/>
+        <child link="wheel_left_link"/>
+        <axis xyz="0 1 0"/>
     </joint>
-    <link name = "caster_front_link">
+    <!-- FRONT CASTER -->
+    <link name="caster_front_link">
         <inertial>
-            <origin xyz="3.89968128948481E-07 2.40073004698083E-07 0.00219173397061506" rpy="0 0 0" />
-            <mass value="1.44379265037903E-06" />
+            <origin xyz="3.89968128948481E-07 2.40073004698083E-07 0.00219173397061506"/>
+            <mass value="1.44379265037903E-06"/>
             <inertia ixx="7.23075276010246E-11" ixy="-6.10956883467859E-16" ixz="2.22849693525031E-15"
-                    iyy="3.8713793085917E-11"  iyz="2.93909858781952E-15"
-                    izz="1.00967486676306E-10" />
+                     iyy="3.8713793085917E-11" iyz="2.93909858781952E-15"
+                     izz="1.00967486676306E-10"/>
         </inertial>
         <visual>
-            <origin rpy = "0 0 0" xyz = "0 0 0"/>
+            <origin xyz="0 0 0" rpy="0 0 0"/>
             <geometry>
-                <mesh filename = "package://bumperbot_description/meshes/caster_front_link.STL"/>
+                <mesh filename="package://bumperbot_description/meshes/caster_front_link.STL"/>
             </geometry>
         </visual>
         <collision>
-            <origin xyz = "0 0 0" rpy = "0 0 0"/>
+            <origin xyz="0 0 0" rpy="0 0 0"/>
             <geometry>
-                <sphere radius = "0.005"/>
+                <sphere radius="0.005"/>
             </geometry>
         </collision>
     </link>
-    <joint name = "caster_front_joint" type = "fixed">
-        <parent link = "base_link"/>
-        <child link = "caster_front_link"/>
-        <origin rpy = "0 0 0" xyz ="0.04755 0 -0.0275"/>
+    <joint name="caster_front_joint" type="fixed">
+        <origin xyz="0.04755 0 -0.0275" rpy="0 0 0"/>
+        <parent link="base_link"/>
+        <child link="caster_front_link"/>
     </joint>
-    <link name = "caster_rear_link">
+    <!-- REAR CASTER (CORREGIDO: antes tenías mal el eje X) -->
+    <link name="caster_rear_link">
         <inertial>
-            <origin xyz="3.8996812895542E-07 2.40073004698083E-07 0.00219173397061509" rpy="0 0 0" />
-            <mass value="1.44379265037902E-06" />
+            <origin xyz="3.8996812895542E-07 2.40073004698083E-07 0.00219173397061509"/>
+            <mass value="1.44379265037902E-06"/>
             <inertia ixx="7.23075276010246E-11" ixy="-6.10956872363424E-16" ixz="2.22849693527207E-15"
-                    iyy="3.87137930859167E-11" iyz="2.939098587861E-15"
-                    izz="1.00967486676306E-10" />
+                     iyy="3.87137930859167E-11" iyz="2.939098587861E-15"
+                     izz="1.00967486676306E-10"/>
         </inertial>
         <visual>
-            <origin rpy = "0 0 0" xyz = "0 0 0"/>
+            <origin xyz="0 0 0" rpy="0 0 0"/>
             <geometry>
-                <mesh filename = "package://bumperbot_description/meshes/caster_rear_link.STL"/>
+                <mesh filename="package://bumperbot_description/meshes/caster_rear_link.STL"/>
             </geometry>
         </visual>
         <collision>
-            <origin xyz = "0 0 0" rpy = "0 0 0"/>
+            <origin xyz="0 0 0" rpy="0 0 0"/>
             <geometry>
-                <sphere radius = "0.033"/>
+                <sphere radius="0.005"/>
             </geometry>
         </collision>
     </link>
-    <joint name = "caster_rear_joint" type = "fixed">
-        <parent link = "base_link"/>
-        <child link = "caster_rear_link"/>
-        <origin rpy = "0 0 0" xyz ="0.04755 0 -0.0275"/>
+    <joint name="caster_rear_joint" type="fixed">
+        <origin xyz="-0.04755 0 -0.0275" rpy="0 0 0"/>
+        <parent link="base_link"/>
+        <child link="caster_rear_link"/>
     </joint>
-    <link name = "can_link">
+    <!-- EXTRA OBJECT (CAN) -->
+    <link name="can_link">
         <visual>
-            <origin xyz="-0.03 0.03 0.0" rpy="1.57 0.0 0.0"/>
+            <origin xyz="-0.03 0.03 0.0" rpy="1.57 0 0"/>
             <geometry>
-                <mesh filename = "package://bumperbot_description/meshes/can.STL"/>
+                <mesh filename="package://bumperbot_description/meshes/can.STL"/>
             </geometry>
         </visual>
     </link>
-    <joint name = "can_joint" type = "fixed">
-        <parent link = "base_link"/>
-        <child link = "can_link"/>
-        <origin rpy = "0 0 0" xyz ="0 0 0.078"/>
+    <joint name="can_joint" type="fixed">
+        <origin xyz="0 0 0.078" rpy="0 0 0"/>
+        <parent link="base_link"/>
+        <child link="can_link"/>
     </joint>
 </robot>

File: Planning/Workspaces/bumperbot_ws/src/bumperbot_description/urdf/bumperbot_gazebo.xacro (robot description, xacro)
@@ -1,37 +1,39 @@
 <?xml version="1.0" encoding="UTF-8"?>
 <robot name = "bumperbot" xmlns:xacro = "http://www.ros.org/wiki/xacro">
-    <gazebo reference = "wheel_right_link">
-        <mu1>100000000000000.0</mu1>
-        <mu2>100000000000000.0</mu2>
+  <!-- Wheels -->
+    <gazebo reference="wheel_left_link">
+        <mu1>1000000000000000.0</mu1>
+        <mu2>1000000000000000.0</mu2>
         <kp>1000000000000.0</kp>
         <kd>10.0</kd>
-        <minDepth> 0.001</minDepth>
+        <minDepth>0.001</minDepth>
         <maxVel>0.1</maxVel>
         <fdir1>1 0 0</fdir1>
     </gazebo>
-    <gazebo reference = "wheel_left_link">
-        <mu1>100000000000000.0</mu1>
-        <mu2>100000000000000.0</mu2>
+    <gazebo reference="wheel_right_link">
+        <mu1>1000000000000000.0</mu1>
+        <mu2>1000000000000000.0</mu2>
         <kp>1000000000000.0</kp>
         <kd>10.0</kd>
-        <minDepth> 0.001</minDepth>
+        <minDepth>0.001</minDepth>
         <maxVel>0.1</maxVel>
         <fdir1>1 0 0</fdir1>
     </gazebo>
-    <gazebo reference = "caster_front_link">
-        <mu1>0.1    </mu1>
+    <!-- Caster Wheels -->
+    <gazebo reference="caster_rear_link">
+        <mu1>0.1</mu1>
         <mu2>0.1</mu2>
         <kp>1000000.0</kp>
         <kd>100.0</kd>
-        <minDepth> 0.001</minDepth>
-        <maxVel>0.1</maxVel>
+        <minDepth>0.001</minDepth>
+        <maxVel>1.0</maxVel>
     </gazebo>
-    <gazebo reference = "caster_rear_link">
-        <mu1>0.1    </mu1>
+    <gazebo reference="caster_front_link">
+        <mu1>0.1</mu1>
         <mu2>0.1</mu2>
         <kp>1000000.0</kp>
         <kd>100.0</kd>
-        <minDepth> 0.001</minDepth>
-        <maxVel>0.1</maxVel>
+        <minDepth>0.001</minDepth>
+        <maxVel>1.0</maxVel>
     </gazebo>
     <gazebo>

Commit message: SLAM with 2D LiDAR

File: Planning/Workspaces/bumperbot_ws/src/bumperbot_description/urdf/bumperbot.urdf.xacro (robot description, xacro)
@@ -116,5 +116,5 @@
         <child link="caster_front_link"/>
     </joint>
-    <!-- REAR CASTER (CORREGIDO: antes tenías mal el eje X) -->
+    <!-- REAR CASTER-->
     <link name="caster_rear_link">
         <inertial>
@@ -144,5 +144,5 @@
     </joint>
     <!-- EXTRA OBJECT (CAN) -->
-    <link name="can_link">
+    <!-- <link name="can_link">
         <visual>
             <origin xyz="-0.03 0.03 0.0" rpy="1.57 0 0"/>
@@ -156,4 +156,23 @@
         <parent link="base_link"/>
         <child link="can_link"/>
+    </joint> -->
+    <link name="laser_link">
+        <visual>
+            <origin xyz="0 0 0" rpy="0 0 0"/>
+            <geometry>
+                <mesh filename="package://bumperbot_description/meshes/laser_link.STL"/>
+            </geometry>
+        </visual>
+        <collision>
+            <origin xyz="0 0 0" rpy="0 0 0"/>
+            <geometry>
+                <mesh filename="package://bumperbot_description/meshes/laser_link.STL"/>
+            </geometry>
+        </collision>
+    </link>
+    <joint name="laser_joint" type="fixed">
+        <parent link="base_link"/>
+        <child link="laser_link"/>
+        <origin xyz="0.0 0.0 0.1208" rpy="0 0 3.14"/>
     </joint>
 </robot>

Commit message: IMU sensor and LiDAR in urdf

File: Planning/Workspaces/bumperbot_ws/src/bumperbot_description/urdf/bumperbot.urdf.xacro (robot description, xacro)
@@ -157,4 +157,31 @@
         <child link="can_link"/>
     </joint> -->
+    <link name="imu_link">
+        <inertial>
+            <origin xyz="-0.00552433659106688 0.000168210391520346 0.000514000497342681" rpy="0 0 0" />
+                <mass value="0.000528415362211671" />
+                <inertia ixx="1.46176048428261E-08" ixy="1.40015117949421E-10" ixz="-1.99633872937403E-12"
+                    iyy="8.59662482954888E-09" iyz="7.52375112767959E-12"
+                    izz="2.30279421279312E-08" />
+        </inertial>
+        <visual>
+            <origin xyz="0 0 0" rpy="0 0 0"/>
+            <geometry>
+                <mesh filename="package://bumperbot_description/meshes/imu_link.STL"/>
+            </geometry>
+        </visual>
+        <collision>
+            <origin xyz="0 0 0" rpy="0 0 0"/>
+            <geometry>
+                <mesh filename="package://bumperbot_description/meshes/imu_link.STL"/>
+            </geometry>
+        </collision>
+    </link>
+    <joint name="imu_joint" type="fixed">
+        <origin xyz="0 0 0.07" rpy="0 0 0"/>
+        <parent link="base_link"/>
+        <child link="imu_link"/>
+        <axis xyz="0 0 0"/>
+    </joint>
     <link name="laser_link">
         <visual>
