Commit message: Robot materials in urdf

File: Planning/Workspaces/bumperbot_ws/src/bumperbot_description/urdf/bumperbot_gazebo.xacro (robot description, xacro)
@@ -1,4 +1,31 @@
 <?xml version="1.0" encoding="UTF-8"?>
-<robot name = "bumperbot" xmlns:xacro = "http://www.ros.org/wiki/xacro">
+<robot name="bumperbot" xmlns:xacro="http://www.ros.org/wiki/xacro">
+    <!-- ========================= -->
+    <!-- MATERIALS -->
+    <!-- ========================= -->
+    <gazebo reference="base_link">
+        <material>Gazebo/DarkRed</material>
+    </gazebo>
+    <gazebo reference="wheel_left_link">
+        <material>Gazebo/FlatBlack</material>
+    </gazebo>
+    <gazebo reference="wheel_right_link">
+        <material>Gazebo/FlatBlack</material>
+    </gazebo>
+    <gazebo reference="caster_front_link">
+        <material>Gazebo/Grey</material>
+    </gazebo>
+    <gazebo reference="caster_rear_link">
+        <material>Gazebo/Grey</material>
+    </gazebo>
+    <gazebo reference="laser_link">
+        <material>Gazebo/Chrome</material>
+    </gazebo>
+    <gazebo reference="imu_link">
+        <material>Gazebo/White</material>
+    </gazebo>
+    <!-- ========================= -->
+    <!-- WHEEL PHYSICS -->
+    <!-- ========================= -->
     <gazebo reference="wheel_left_link">
         <mu1>1000000000000000.0</mu1>
@@ -35,26 +62,42 @@
         <maxVel>1.0</maxVel>
     </gazebo>
+    <!-- ========================= -->
+    <!-- ROS2 CONTROL + SENSORS -->
+    <!-- ========================= -->
     <gazebo>
-        <xacro:if value = "$(arg is_ignition)">
-            <plugin filename="gz_ros2_control-system" name="gz_ros2_control::GazeboSimROS2ControlPlugin">
-                <parameters>$(find bumperbot_controller)/config/bumperbot_controllers.yaml</parameters>
+        <xacro:if value="$(arg is_ignition)">
+            <plugin filename="gz_ros2_control-system"
+                    name="gz_ros2_control::GazeboSimROS2ControlPlugin">
+                <parameters>
+                    $(find bumperbot_controller)/config/bumperbot_controllers.yaml
+                </parameters>
             </plugin>
-            <plugin filename="libignition-gazebo-imu-system.so" name="ignition::gazebo::systems::Imu">
+            <plugin filename="libignition-gazebo-imu-system.so"
+                    name="ignition::gazebo::systems::Imu">
             </plugin>
-            <plugin filename="libignition-gazebo-sensors-system.so" name="ignition::gazebo::systems::Sensors">
+            <plugin filename="libignition-gazebo-sensors-system.so"
+                    name="ignition::gazebo::systems::Sensors">
                 <render_engine>ogre2</render_engine>
             </plugin>
         </xacro:if>
-        <xacro:unless value = "$(arg is_ignition)">
-            <plugin filename="gz_ros2_control-system" name="gz_ros2_control::GazeboSimROS2ControlPlugin">
-                <parameters>$(find bumperbot_controller)/config/bumperbot_controllers.yaml</parameters>
+        <xacro:unless value="$(arg is_ignition)">
+            <plugin filename="gz_ros2_control-system"
+                    name="gz_ros2_control::GazeboSimROS2ControlPlugin">
+                <parameters>
+                    $(find bumperbot_controller)/config/bumperbot_controllers.yaml
+                </parameters>
             </plugin>
-            <plugin filename="gz-sim-imu-system" name="gz::sim::systems::Imu">
+            <plugin filename="gz-sim-imu-system"
+                    name="gz::sim::systems::Imu">
             </plugin>
-            <plugin filename="gz-sim-sensors-system" name="gz::sim::systems::Sensors">
+            <plugin filename="gz-sim-sensors-system"
+                    name="gz::sim::systems::Sensors">
                 <render_engine>ogre2</render_engine>
             </plugin>
         </xacro:unless>
     </gazebo>
+    <!-- ========================= -->
+    <!-- IMU -->
+    <!-- ========================= -->
     <gazebo reference="imu_link">
         <sensor name="imu" type="imu">
@@ -107,4 +150,7 @@
         </sensor>
     </gazebo>
+    <!-- ========================= -->
+    <!-- LIDAR -->
+    <!-- ========================= -->
     <gazebo reference="laser_link">
         <sensor name="lidar" type="gpu_ray">

Commit message: Robot materials in urdf

File: Planning/Workspaces/bumperbot_ws/src/bumperbot_description/urdf/bumperbot_gazebo.xacro (robot description, xacro)
@@ -5,17 +5,17 @@
     <!-- ========================= -->
     <gazebo reference="base_link">
-        <material>Gazebo/DarkRed</material>
+        <material>Gazebo/Red</material>
     </gazebo>
     <gazebo reference="wheel_left_link">
-        <material>Gazebo/FlatBlack</material>
+        <material>Gazebo/Black</material>
     </gazebo>
     <gazebo reference="wheel_right_link">
-        <material>Gazebo/FlatBlack</material>
+        <material>Gazebo/Black</material>
     </gazebo>
     <gazebo reference="caster_front_link">
-        <material>Gazebo/Grey</material>
+        <material>Gazebo/White</material>
     </gazebo>
     <gazebo reference="caster_rear_link">
-        <material>Gazebo/Grey</material>
+        <material>Gazebo/White</material>
     </gazebo>
     <gazebo reference="laser_link">
@@ -23,5 +23,5 @@
     </gazebo>
     <gazebo reference="imu_link">
-        <material>Gazebo/White</material>
+        <material>Gazebo/Grey</material>
     </gazebo>
     <!-- ========================= -->
